File: Kicad_files/IronControllerHardware/IronControllerHardware.kicad_sch (KiCad schematic)
At the start: 16 parts

Commit message: update schematics
Parts:
- R? (x2): value 3.3K -> 1K
Connections:
- net 0: now also J?.1 (Pin_1), J?.1 (Pin_1); no longer R?.2, R?.2
- new net: R?.1, R?.1, U?.9 (3.3)
- new net: J?.2 (Pin_2), R?.2, R?.2
- new net: J?.2 (Pin_2), R?.1, R?.2
Other:
- moved on the sheet: J?, R?

Commit message: implement debug mode
Parts:
- removed R?: 22K, symbol Device:R
- added J3: Screw_Terminal_01x02, symbol Connector:Screw_Terminal_01x02
- added J?: Conn_01x02_Male, symbol Connector:Conn_01x02_Male
- added Q1: IRF3808, Package_TO_SOT_THT:TO-220-3_Vertical, symbol Transistor_FET:IPP060N06N
- added Q3, Q?: BSS138, Package_TO_SOT_SMD:SOT-23, symbol Transistor_FET:2N7000
- added R6: 2.2K, symbol Device:R
- added R? (x2): 22K, symbol Device:R
- Q2: renamed from Q?; value IPP060N06N -> IRF3808
- Q4: renamed from Q?; value 2N7000 -> BSS138; footprint Package_TO_SOT_THT:TO-92_Inline -> Package_TO_SOT_SMD:SOT-23
- gave numbers to parts that had none: 13
Connections:
- net 0: now also Q1.3 (S), Q?.1 (S), R6.1
- net 5V: now also J?.2 (Pin_2), R?.1, R?.1
- net at J1.2 (Pin_2), J2.2 (Pin_2), PWR1.1 (In): now also J3.2 (Pin_2)
- net at Q2.1 (G), Q4.3 (D): now also R?.2
- net at U1.18: now also Q?.2 (G)
- net at U1.5: now also Q3.2 (G)
- new net: Q3.1 (S), R6.2
- new net: Q1.1 (G), Q3.3 (D), R?.2
- new net: J?.1 (Pin_1), Q?.3 (D)
- new net: J3.1 (Pin_1), Q1.2 (D)
Other:
- company: (none) -> jose luu
- title: (none) -> Lisa's iron
- moved on the sheet: R7

Commit message: fixes
Parts:
- gave numbers to parts that had none: 4
Connections:
- net at Q3.1 (S), R6.2: now also U1.5
- net at Q3.2 (G): now also Q4.2 (G), U1.11 (3.3); no longer U1.5
Other:
- moved on the sheet: C1, Q3, Q5, R2, R4

Commit message: mise a jour schema, corrrection bugs
Parts:
- added U?: AMS1117-5.0, Package_TO_SOT_SMD:SOT-223-3_TabPin2, symbol Regulator_Linear:AMS1117-5.0
- Q1, Q2: value IRF3808 -> IRFB3206
- R1, R2: value 1K -> 3.9K
Connections:
- net 0: now also U?.1 (GND)
- net 5V: now also U?.2 (VO); no longer PWR1.2 (Out), R5.1, R8.1
- new net 10.5V: PWR1.2 (Out), R5.1, R8.1, U?.3 (VI)
Changed lines of the file:
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@@
   (junction (at 92.71 60.96) (diameter 0) (color 0 0 0 0)
   )
+  (junction (at 100.33 38.1) (diameter 0) (color 0 0 0 0)
+  )
   (junction (at 66.04 124.46) (diameter 0) (color 0 0 0 0)
   )
-  (junction (at 100.33 38.1) (diameter 0) (color 0 0 0 0)
-  )
   (junction (at 38.1 41.91) (diameter 0) (color 0 0 0 0)
   )
+  (wire (pts (xy 100.33 38.1) (xy 107.95 38.1))
+    (stroke (width 0) (type default) (color 0 0 0 0))
+  )
   (wire (pts (xy 130.81 38.1) (xy 130.81 86.36))
     (stroke (width 0) (type default) (color 0 0 0 0))
@@
     (stroke (width 0) (type default) (color 0 0 0 0))
   )
-  (wire (pts (xy 100.33 38.1) (xy 130.81 38.1))
-    (stroke (width 0) (type default) (color 0 0 0 0))
-  )
   (wire (pts (xy 43.18 128.27) (xy 43.18 140.97))
     (stroke (width 0) (type default) (color 0 0 0 0))
@@
     (stroke (width 0) (type default) (color 0 0 0 0))
   )
+  (wire (pts (xy 123.19 38.1) (xy 130.81 38.1))
+    (stroke (width 0) (type default) (color 0 0 0 0))
+  )
   (wire (pts (xy 142.24 97.79) (xy 142.24 88.9))
     (stroke (width 0) (type default) (color 0 0 0 0))
@@
     (stroke (width 0) (type default) (color 0 0 0 0))
   )
+  (wire (pts (xy 115.57 45.72) (xy 115.57 48.26))
+    (stroke (width 0) (type default) (color 0 0 0 0))
+  )
   (wire (pts (xy 92.71 38.1) (xy 92.71 44.45))
     (stroke (width 0) (type default) (color 0 0 0 0))
@@
     (stroke (width 0) (type default) (color 0 0 0 0))
   )
-  (label "5V" (at 114.3 38.1 0)
-    (effects (font (size 1.27 1.27)) (justify left bottom))
+  (global_label "5V" (shape input) (at 139.7 38.1 0) (fields_autoplaced)
+    (effects (font (size 1.27 1.27)) (justify left))
+    (property "Intersheet References" "${INTERSHEET_REFS}" (id 0) (at 144.4112 38.0206 0)
+      (effects (font (size 1.27 1.27)) (justify left) hide)
+    )
+  )
+  (global_label "10.5V" (shape input) (at 88.9 38.1 90) (fields_autoplaced)
+    (effects (font (size 1.27 1.27)) (justify left))
+    (property "Intersheet References" "${INTERSHEET_REFS}" (id 0) (at 88.8206 30.365 90)
+      (effects (font (size 1.27 1.27)) (justify left) hide)
+    )
   )
   (symbol (lib_id "Connector:Screw_Terminal_01x02") (at 30.48 62.23 180) (unit 1)
@@
       (effects (font (size 1.27 1.27)) (justify left))
     )
-    (property "Value" "1K" (id 1) (at 48.26 147.32 0)
+    (property "Value" "3.9K" (id 1) (at 48.26 147.32 0)
       (effects (font (size 1.27 1.27)) (justify left))
     )
@@
       (effects (font (size 1.27 1.27)) (justify left))
     )
-    (property "Value" "IRF3808" (id 1) (at 67.31 62.23 0)
+    (property "Value" "IRFB3206" (id 1) (at 67.31 62.23 0)
       (effects (font (size 1.27 1.27)) (justify left))
     )
@@
       (effects (font (size 1.27 1.27)) (justify left))
     )
-    (property "Value" "1K" (id 1) (at 48.26 133.35 0)
+    (property "Value" "3.9K" (id 1) (at 48.26 133.35 0)
       (effects (font (size 1.27 1.27)) (justify left))
     )
@@
     (pin "1")
     (pin "2")
+  )
+  (symbol (lib_id "Regulator_Linear:AMS1117-5.0") (at 115.57 38.1 0) (unit 1)
+    (in_bom yes) (on_board yes) (fields_autoplaced)
+    (property "Reference" "U?" (id 0) (at 115.57 30.48 0))
+    (property "Value" "AMS1117-5.0" (id 1) (at 115.57 33.02 0))
+    (property "Footprint" "Package_TO_SOT_SMD:SOT-223-3_TabPin2" (id 2) (at 115.57 33.02 0)
+      (effects (font (size 1.27 1.27)) hide)
+    )
+    (property "Datasheet" "http://www.advanced-monolithic.com/pdf/ds1117.pdf" (id 3) (at 118.11 44.45 0)
+      (effects (font (size 1.27 1.27)) hide)
+    )
+    (pin "1")
+    (pin "2")
+    (pin "3")
+  )
+  (symbol (lib_id "pspice:0") (at 115.57 48.26 0) (unit 1)
+    (in_bom yes) (on_board yes) (fields_autoplaced)
+    (property "Reference" "#GND?" (id 0) (at 115.57 50.8 0)
+      (effects (font (size 1.27 1.27)) hide)
+    )
+    (property "Value" "0" (id 1) (at 115.57 45.72 0))
+    (property "Footprint" "" (id 2) (at 115.57 48.26 0)
+      (effects (font (size 1.27 1.27)) hide)
+    )
+    (property "Datasheet" "~" (id 3) (at 115.57 48.26 0)
+      (effects (font (size 1.27 1.27)) hide)
+    )
+    (pin "1")
   )
   (symbol (lib_id "pspice:0") (at 168.91 134.62 0) (unit 1)
@@
       (effects (font (size 1.27 1.27)) (justify left))
     )
-    (property "Value" "IRF3808" (id 1) (at 55.88 74.93 0)
+    (property "Value" "IRFB3206" (id 1) (at 55.88 74.93 0)
       (effects (font (size 1.27 1.27)) (justify left))
     )
@@
       (reference "#GND09") (unit 1) (value "0") (footprint "")
     )
+    (path "/960e876b-e4ea-4e29-9683-beb7d916433e"
+      (reference "#GND?") (unit 1) (value "0") (footprint "")
+    )
     (path "/2f445251-dc99-4305-95e3-8cf5e7907216"
       (reference "C1") (unit 1) (value "4.7u") (footprint "")
@@
     )
     (path "/f932a143-fd0f-4b5c-9490-8098723d9770"
-      (reference "Q1") (unit 1) (value "IRF3808") (footprint "Package_TO_SOT_THT:TO-220-3_Vertical")
+      (reference "Q1") (unit 1) (value "IRFB3206") (footprint "Package_TO_SOT_THT:TO-220-3_Vertical")
     )
     (path "/6452710d-466d-4f81-84a7-9b2459a2e1f3"
-      (reference "Q2") (unit 1) (value "IRF3808") (footprint "Package_TO_SOT_THT:TO-220-3_Vertical")
+      (reference "Q2") (unit 1) (value "IRFB3206") (footprint "Package_TO_SOT_THT:TO-220-3_Vertical")
     )
     (path "/9bd8ef1d-532a-4927-afe5-162e6702eed1"
@@
     )
     (path "/8f574603-49f5-4e31-b11b-c6ba7d1b30ca"
-      (reference "R1") (unit 1) (value "1K") (footprint "")
+      (reference "R1") (unit 1) (value "3.9K") (footprint "")
     )
     (path "/2678dfd5-a23c-4965-ae6f-de8211b6dd15"
-      (reference "R2") (unit 1) (value "1K") (footprint "")
+      (reference "R2") (unit 1) (value "3.9K") (footprint "")
     )
     (path "/5bfde62b-ec06-4460-8a4a-22484098f631"
@@
       (reference "U1") (unit 1) (value "Heltec_HTIT-WB32") (footprint "")
     )
-  )
+    (path "/8f7fe4c8-3d1e-44b7-a053-1c37b539385b"
+      (reference "U?") (unit 1) (value "AMS1117-5.0") (footprint "Package_TO_SOT_SMD:SOT-223-3_TabPin2")
+    )
+  )
